File: board_files/MIPI_interface_board.kicad_pcb (KiCad board)
At the start: 2 copper layers, 167.6 x 95.2 mm, 20 parts, among them U1 Pico, X1 CONBNC002, X2 CONBNC002, X3 CONBNC002, X4 CONBNC002, X5 CONBNC002

Commit message: completed README and added corrected versions of board files (no trace rounding)
Routing:
- net +3.3V: track 321.2 -> 325.5 mm
- net /SDATA_MAIN: track 181.9 -> 183.8 mm
- net /SDA_OUT: track 149.3 -> 151.1 mm
- net /SCLK_MAIN: track 182.4 -> 184.0 mm
- net Net-(A1-Pad10): track 41.8 -> 42.8 mm
- net Net-(A1-Pad9): track 41.8 -> 42.8 mm
- net Net-(A1-Pad16): track 62.4 -> 63.0 mm
- net /SCL_OUT: track 26.9 -> 27.4 mm
- net /VCC_OUT: track 14.4 -> 14.9 mm
Other:
- board text added: "GBT"
